File: BT66B_RJ45_JB.kicad_pcb (KiCad board)
At the start: 2 copper layers, 95.5 x 41.3 mm, 9 parts, among them J1 RJ45, J2 RJ45, J3 RJ45, J4 RJ45, J5 RJ45

Commit message: Latest changes
Routing:
- net /L4+: track 72.1 -> 91.8 mm, vias 0 -> 1
- net /L1-: track 15.3 -> 32.3 mm
- net /L2-: track 22.6 -> 39.2 mm, vias 1 -> 0
- net /L2+: track 23.3 -> 37.7 mm, vias 0 -> 1
- net /L4-: track 79.4 -> 92.2 mm, vias 0 -> 1
- net /L1+: track 19.9 -> 25.4 mm, vias 0 -> 2
- net /L3+: track 43.2 -> 46.7 mm
Other:
- board text added: "JLCJLCJLCJLC"
- board text added: "https://github.com/cu-telecom/BT66B_RJ45_JB v0.3"
- board text removed: "https://github.com/cu-telecom/BT66B_RJ45_JB v0.1"
